File: Fury-Taur.kicad_sch (KiCad schematic)
At the start: 26 parts, among them J1 Pickup, J2 Audio Out, Q1 J201, Q2 J201, SW1 Push Pull, SW2 SW_SPDT

Commit message: Added components to PCB board
Parts:
- C1, C2, C3, C4, C6, C7: footprint (none) -> Capacitor_THT:C_Disc_D14.5mm_W5.0mm_P10.00mm
- D1: footprint (none) -> digikey-footprints:Diode_DO-35_P10mm
- D2, D3: footprint digikey-footprints:DO-35 -> digikey-footprints:DO-41
- SW2: footprint (none) -> Button_Switch_THT:SW_Slide_SPDT_Straight_CK_OS102011MS2Q
Changed lines of the file:
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@@
 			)
 		)
-		(property "Footprint" ""
+		(property "Footprint" "digikey-footprints:Diode_DO-35_P10mm"
 			(at 143.51 76.2 0)
 			(hide yes)
@@
 			)
 		)
-		(property "Footprint" ""
+		(property "Footprint" "Capacitor_THT:C_Disc_D14.5mm_W5.0mm_P10.00mm"
 			(at 136.8552 90.17 0)
 			(hide yes)
@@
 			)
 		)
-		(property "Footprint" "digikey-footprints:DO-35"
+		(property "Footprint" "digikey-footprints:DO-41"
 			(at 172.72 129.54 0)
 			(hide yes)
@@
 			)
 		)
-		(property "Footprint" ""
+		(property "Footprint" "Capacitor_THT:C_Disc_D14.5mm_W5.0mm_P10.00mm"
 			(at 110.49 110.1852 0)
 			(hide yes)
@@
 			)
 		)
-		(property "Footprint" ""
+		(property "Footprint" "Button_Switch_THT:SW_Slide_SPDT_Straight_CK_OS102011MS2Q"
 			(at 177.8 116.84 0)
 			(hide yes)
@@
 			)
 		)
-		(property "Footprint" ""
+		(property "Footprint" "Capacitor_THT:C_Disc_D14.5mm_W5.0mm_P10.00mm"
 			(at 122.8852 90.17 0)
 			(hide yes)
@@
 			)
 		)
-		(property "Footprint" "digikey-footprints:DO-35"
+		(property "Footprint" "digikey-footprints:DO-41"
 			(at 176.53 129.54 0)
 			(hide yes)
@@
 			)
 		)
-		(property "Footprint" ""
+		(property "Footprint" "Capacitor_THT:C_Disc_D14.5mm_W5.0mm_P10.00mm"
 			(at 173.6852 90.17 0)
 			(hide yes)
@@
 			)
 		)
-		(property "Footprint" ""
+		(property "Footprint" "Capacitor_THT:C_Disc_D14.5mm_W5.0mm_P10.00mm"
 			(at 160.02 103.8352 0)
 			(hide yes)
@@
 			)
 		)
-		(property "Footprint" ""
+		(property "Footprint" "Capacitor_THT:C_Disc_D14.5mm_W5.0mm_P10.00mm"
 			(at 130.81 106.3752 0)
 			(hide yes)

Commit message: Rearranged PCB, added footprints
Parts:
- removed R1, R5: 20K, Resistor_THT:R_Axial_DIN0411_L9.9mm_D3.6mm_P12.70mm_Horizontal, symbol Device:R_Trim
- added J2: Output, TerminalBlock_4Ucon:TerminalBlock_4Ucon_1x03_P3.50mm_Horizontal, symbol Connector:Screw_Terminal_01x03
- added RV2, RV3: 20K, Potentiometer_THT:Potentiometer_Bourns_3296W_Vertical, symbol Device:R_Potentiometer_Trim_US
- C1, C4, C6: footprint Capacitor_THT:C_Disc_D14.5mm_W5.0mm_P10.00mm -> Capacitor_THT:C_Disc_D7.0mm_W2.5mm_P5.00mm
- C2, C7: footprint Capacitor_THT:C_Disc_D14.5mm_W5.0mm_P10.00mm -> Capacitor_THT:C_Disc_D5.1mm_W3.2mm_P5.00mm
- C3: footprint Capacitor_THT:C_Disc_D14.5mm_W5.0mm_P10.00mm -> Capacitor_THT:C_Disc_D5.0mm_W2.5mm_P5.00mm
- C5: footprint (none) -> Capacitor_THT:C_Radial_D6.3mm_H11.0mm_P2.50mm
- J1: footprint (none) -> TerminalBlock_4Ucon:TerminalBlock_4Ucon_1x05_P3.50mm_Horizontal
- R2: renamed from R3; footprint (none) -> Resistor_THT:R_Axial_DIN0204_L3.6mm_D1.6mm_P7.62mm_Horizontal
- R3: renamed from R4; footprint Potentiometer_THT:Potentiometer_Runtron_RM-065_Vertical -> Potentiometer_THT:Potentiometer_Bourns_3296W_Vertical
- R5: renamed from R7; footprint Potentiometer_THT:Potentiometer_Runtron_RM-065_Vertical -> Potentiometer_THT:Potentiometer_Bourns_3296W_Vertical
- renumbered J2 to J3, R2 to R1, R6 to R4
Connections:
- net BAT -: now also J3.R, J2.2 (Pin_2); no longer J3.S
- net at C6.2, C7.2, Q2.1 (D): now also RV3.3
- net at J3.T, SW1.5 (B): now also J2.1 (Pin_1)
- net at C2.2, C3.2, Q1.1 (D): now also RV2.3
- new net: C2.1, C4.1, C5.1, C7.1, D1.1 (K), RV2.1, RV2.2, RV3.1, RV3.2
- new net: D2.1 (K), D3.2 (A), J2.3 (Pin_3), J3.S, Q1.2 (S), Q2.2 (S), R1.2, R3.3, R5.3, RV1.3
- new net: C1.1, Q1.3 (G), R1.1
- no-connect marks 0 -> 1
Other:
- moved on the sheet: C2, J3, R1

Commit message: Rearranged PCB, added footprints, sanity checked net q
Other:
- moved on the sheet: J2, J3
Changed lines of the file:
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@@
 	(paper "A4")
 	(junction
-		(at 210.82 148.59)
+		(at 195.58 146.05)
+		(diameter 0)
+		(color 0 0 0 0)
+	)
+	(junction
+		(at 210.82 140.97)
 		(diameter 0)
 		(color 0 0 0 0)
@@
 	)
 	(junction
-		(at 195.58 146.05)
+		(at 173.99 146.05)
+		(diameter 0)
+		(color 0 0 0 0)
+	)
+	(junction
+		(at 165.1 92.71)
+		(diameter 0)
+		(color 0 0 0 0)
+	)
+	(junction
+		(at 118.11 146.05)
+		(diameter 0)
+		(color 0 0 0 0)
+	)
+	(junction
+		(at 182.88 102.87)
+		(diameter 0)
+		(color 0 0 0 0)
+	)
+	(junction
+		(at 82.55 102.87)
 		(diameter 0)
 		(color 0 0 0 0)
@@
 	)
 	(junction
-		(at 173.99 146.05)
-		(diameter 0)
-		(color 0 0 0 0)
-	)
-	(junction
-		(at 165.1 92.71)
-		(diameter 0)
-		(color 0 0 0 0)
-	)
-	(junction
-		(at 118.11 146.05)
-		(diameter 0)
-		(color 0 0 0 0)
-	)
-	(junction
-		(at 182.88 102.87)
-		(diameter 0)
-		(color 0 0 0 0)
-	)
-	(junction
-		(at 82.55 102.87)
+		(at 147.32 82.55)
 		(diameter 0)
 		(color 0 0 0 0)
@@
 	(junction
 		(at 210.82 146.05)
-		(diameter 0)
-		(color 0 0 0 0)
-	)
-	(junction
-		(at 147.32 82.55)
 		(diameter 0)
 		(color 0 0 0 0)
@@
 	(wire
 		(pts
-			(xy 195.58 148.59) (xy 195.58 146.05)
-		)
-		(stroke
-			(width 0)
-			(type default)
-		)
-	)
-	(wire
-		(pts
-			(xy 241.3 148.59) (xy 210.82 148.59)
+			(xy 241.3 146.05) (xy 210.82 146.05)
 		)
 		(stroke
@@
 	(wire
 		(pts
-			(xy 210.82 146.05) (xy 241.3 146.05)
+			(xy 210.82 143.51) (xy 241.3 143.51)
 		)
 		(stroke
@@
 	(wire
 		(pts
-			(xy 199.39 146.05) (xy 210.82 146.05)
+			(xy 199.39 143.51) (xy 210.82 143.51)
 		)
 		(stroke
@@
 	(wire
 		(pts
-			(xy 109.22 143.51) (xy 210.82 143.51)
-		)
-		(stroke
-			(width 0)
-			(type default)
-		)
-	)
-	(wire
-		(pts
-			(xy 199.39 146.05) (xy 199.39 152.4)
+			(xy 109.22 140.97) (xy 210.82 140.97)
 		)
 		(stroke
@@
 	(wire
 		(pts
-			(xy 210.82 143.51) (xy 241.3 143.51)
+			(xy 210.82 140.97) (xy 241.3 140.97)
 		)
 		(stroke
@@
 	(wire
 		(pts
-			(xy 109.22 121.92) (xy 109.22 143.51)
+			(xy 109.22 121.92) (xy 109.22 140.97)
 		)
 		(stroke
@@
 	(wire
 		(pts
-			(xy 210.82 148.59) (xy 195.58 148.59)
+			(xy 199.39 143.51) (xy 199.39 152.4)
+		)
+		(stroke
+			(width 0)
+			(type default)
+		)
+	)
+	(wire
+		(pts
+			(xy 210.82 146.05) (xy 195.58 146.05)
 		)
 		(stroke
@@
 	(symbol
 		(lib_id "Connector:Screw_Terminal_01x03")
-		(at 215.9 146.05 0)
+		(at 215.9 143.51 0)
 		(unit 1)
 		(body_style 1)
@@
 		(fields_autoplaced yes)
 		(property "Reference" "J2"
+			(at 218.44 142.2399 0)
+			(show_name no)
+			(do_not_autoplace no)
+			(effects
+				(font
+					(size 1.27 1.27)
+				)
+				(justify left)
+			)
+		)
+		(property "Value" "Output"
 			(at 218.44 144.7799 0)
 			(show_name no)
@@
 			)
 		)
-		(property "Value" "Output"
-			(at 218.44 147.3199 0)
-			(show_name no)
-			(do_not_autoplace no)
-			(effects
-				(font
-					(size 1.27 1.27)
-				)
-				(justify left)
-			)
-		)
 		(property "Footprint" "TerminalBlock_4Ucon:TerminalBlock_4Ucon_1x03_P3.50mm_Horizontal"
-			(at 215.9 146.05 0)
+			(at 215.9 143.51 0)
 			(hide yes)
 			(show_name no)
@@
 		)
 		(property "Datasheet" ""
-			(at 215.9 146.05 0)
+			(at 215.9 143.51 0)
 			(hide yes)
 			(show_name no)
@@
 		)
 		(property "Description" "Generic screw terminal, single row, 01x03, script generated (kicad-library-utils/schlib/autogen/connector/)"
-			(at 215.9 146.05 0)
+			(at 215.9 143.51 0)
 			(hide yes)
 			(show_name no)
@@
 	(symbol
 		(lib_id "Connector_Audio:AudioJack3")
-		(at 246.38 146.05 180)
+		(at 246.38 143.51 180)
 		(unit 1)
 		(body_style 1)
@@
 		(fields_autoplaced yes)
 		(property "Reference" "J3"
+			(at 254 141.6049 0)
+			(show_name no)
+			(do_not_autoplace no)
+			(effects
+				(font
+					(size 1.27 1.27)
+				)
+				(justify right)
+			)
+		)
+		(property "Value" "Audio Out"
 			(at 254 144.1449 0)
 			(show_name no)
@@
 			)
 		)
-		(property "Value" "Audio Out"
-			(at 254 146.6849 0)
-			(show_name no)
-			(do_not_autoplace no)
-			(effects
-				(font
-					(size 1.27 1.27)
-				)
-				(justify right)
-			)
-		)
 		(property "Footprint" ""
-			(at 246.38 146.05 0)
+			(at 246.38 143.51 0)
 			(hide yes)
 			(show_name no)
@@
 		)
 		(property "Datasheet" ""
-			(at 246.38 146.05 0)
+			(at 246.38 143.51 0)
 			(hide yes)
 			(show_name no)
@@
 		)
 		(property "Description" "Audio Jack, 3 Poles (Stereo / TRS)"
-			(at 246.38 146.05 0)
-			(hide yes)
-			(show_name no)
+			(at 246.38 143.51 0)
+			(hide yes)
+			(show_name no)

Commit message: Updated Silkscreens
Connections:
- net GND: now also D2.1 (K), D3.2 (A), J2.3 (Pin_3), J3.S, Q1.2 (S), Q2.2 (S), R1.2, R3.3, R5.3, RV1.3
Changed lines of the file:
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@@
+	)
+	(junction
+		(at 88.9 146.05)
+		(diameter 0)
+		(color 0 0 0 0)
 	)
 	(junction
@@
 					(unit 1)
 				)
+			)
+		)
+	)
+	(symbol
+		(lib_id "power:GND")
+		(at 88.9 146.05 0)
+		(unit 1)
+		(body_style 1)
+		(exclude_from_sim no)
+		(in_bom yes)
+		(on_board yes)
+		(in_pos_files yes)
+		(dnp no)
+		(fields_autoplaced yes)
+		(property "Reference" "#PWR06"
+			(at 88.9 152.4 0)
+			(hide yes)
+			(show_name no)
+			(do_not_autoplace no)
+			(effects
+				(font
+					(size 1.27 1.27)
+				)
+			)
+		)
+		(property "Value" "GND"
+			(at 88.9 151.13 0)
+			(show_name no)
+			(do_not_autoplace no)
+			(effects
+				(font
+					(size 1.27 1.27)
+				)
+			)
+		)
+		(property "Footprint" ""
+			(at 88.9 146.05 0)
+			(hide yes)
+			(show_name no)
+			(do_not_autoplace no)
+			(effects
+				(font
+					(size 1.27 1.27)
+				)
+			)
+		)
+		(property "Datasheet" ""
+			(at 88.9 146.05 0)
+			(hide yes)
+			(show_name no)
+			(do_not_autoplace no)
+			(effects
+				(font
+					(size 1.27 1.27)
+				)
+			)
+		)
+		(property "Description" "Power symbol creates a global label with name \"GND\" , ground"
+			(at 88.9 146.05 0)
+			(hide yes)
+			(show_name no)
+			(do_not_autoplace no)
+			(effects
+				(font
+					(size 1.27 1.27)
+				)
+			)
+		)
+		(pin "1"
+		)
+		(instances
+			(project "Fury-Taur"
+				(path "/9aaae789-b710-4a8a-aadd-535a824b9702"
+					(reference "#PWR06")
+					(unit 1)
+				)

Commit message: Changed footprints for Diodes
Parts:
- D1: footprint digikey-footprints:Diode_DO-35_P10mm -> Diode_THT:D_DO-35_SOD27_P10.16mm_Horizontal
- D2, D3: footprint digikey-footprints:DO-41 -> Diode_THT:D_DO-41_SOD81_P10.16mm_Horizontal
Changed lines of the file:
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@@
 			)
 		)
-		(property "Footprint" "digikey-footprints:Diode_DO-35_P10mm"
+		(property "Footprint" "Diode_THT:D_DO-35_SOD27_P10.16mm_Horizontal"
 			(at 143.51 76.2 0)
 			(hide yes)
@@
 			)
 		)
-		(property "Footprint" "digikey-footprints:DO-41"
+		(property "Footprint" "Diode_THT:D_DO-41_SOD81_P10.16mm_Horizontal"
 			(at 172.72 129.54 0)
 			(hide yes)
@@
 			)
 		)
-		(property "Footprint" "digikey-footprints:DO-41"
+		(property "Footprint" "Diode_THT:D_DO-41_SOD81_P10.16mm_Horizontal"
 			(at 176.53 129.54 0)
 			(hide yes)

Commit message: Adjusted bias pots
Connections:
- net at C2.1, C4.1, C5.1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: now also RV2.3, RV3.3; no longer RV2.1, RV3.1
- net at C6.2, C7.2, Q2.1 (D): now also RV3.1; no longer RV3.3
- net at C2.2, C3.2, Q1.1 (D): now also RV2.1; no longer RV2.3
Changed lines of the file:
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@@
 	)
 	(symbol
+		(lib_name "R_Potentiometer_Trim_US_1")
 		(lib_id "Device:R_Potentiometer_Trim_US")
 		(at 115.57 86.36 0)
@@
 	)
 	(symbol
+		(lib_name "R_Potentiometer_Trim_US_2")
 		(lib_id "Device:R_Potentiometer_Trim_US")
 		(at 165.1 86.36 0)

Commit message: Removed C4, adjusted c5 to 100uf from 220uf
Parts:
- removed C4: 100nf, Capacitor_THT:C_Disc_D7.0mm_W2.5mm_P5.00mm, symbol Device:C
- C5: value 220uf -> 100uf
Changed lines of the file:
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@@
-	)
-	(junction
-		(at 135.89 82.55)
-		(diameter 0)
-		(color 0 0 0 0)
 	)
 	(junction
@@
 	)
 	(junction
-		(at 147.32 90.17)
-		(diameter 0)
-		(color 0 0 0 0)
-	)
-	(junction
 		(at 119.38 82.55)
 		(diameter 0)
@@
 	(wire
 		(pts
-			(xy 123.19 82.55) (xy 135.89 82.55)
-		)
-		(stroke
-			(width 0)
-			(type default)
-		)
-	)
-	(wire
-		(pts
-			(xy 135.89 90.17) (xy 147.32 90.17)
-		)
-		(stroke
-			(width 0)
-			(type default)
-		)
-	)
-	(wire
-		(pts
 			(xy 60.96 96.52) (xy 74.93 96.52)
 		)
@@
 	(wire
 		(pts
-			(xy 135.89 82.55) (xy 147.32 82.55)
+			(xy 123.19 82.55) (xy 147.32 82.55)
 		)
 		(stroke
@@
 				(path "/9aaae789-b710-4a8a-aadd-535a824b9702"
 					(reference "J2")
-					(unit 1)
-				)
-			)
-		)
-	)
-	(symbol
-		(lib_id "Device:C")
-		(at 135.89 86.36 0)
-		(unit 1)
-		(body_style 1)
-		(exclude_from_sim no)
-		(in_bom yes)
-		(on_board yes)
-		(in_pos_files yes)
-		(dnp no)
-		(fields_autoplaced yes)
-		(property "Reference" "C4"
-			(at 139.7 85.0899 0)
-			(show_name no)
-			(do_not_autoplace no)
-			(effects
-				(font
-					(size 1.27 1.27)
-				)
-				(justify left)
-			)
-		)
-		(property "Value" "100nf"
-			(at 139.7 87.6299 0)
-			(show_name no)
-			(do_not_autoplace no)
-			(effects
-				(font
-					(size 1.27 1.27)
-				)
-				(justify left)
-			)
-		)
-		(property "Footprint" "Capacitor_THT:C_Disc_D7.0mm_W2.5mm_P5.00mm"
-			(at 136.8552 90.17 0)
-			(hide yes)
-			(show_name no)
-			(do_not_autoplace no)
-			(effects
-				(font
-					(size 1.27 1.27)
-				)
-			)
-		)
-		(property "Datasheet" ""
-			(at 135.89 86.36 0)
-			(hide yes)
-			(show_name no)
-			(do_not_autoplace no)
-			(effects
-				(font
-					(size 1.27 1.27)
-				)
-			)
-		)
-		(property "Description" "Unpolarized capacitor"
-			(at 135.89 86.36 0)
-			(hide yes)
-			(show_name no)
-			(do_not_autoplace no)
-			(effects
-				(font
-					(size 1.27 1.27)
-				)
-			)
-		)
-		(pin "1"
-		)
-		(pin "2"
-		)
-		(instances
-			(project "Fury-Taur"
-				(path "/9aaae789-b710-4a8a-aadd-535a824b9702"
-					(reference "C4")
 					(unit 1)
 				)
@@
 			)
 		)
-		(property "Value" "220uf"
+		(property "Value" "100uf"
 			(at 151.13 87.8839 0)
 			(show_name no)

Commit message: Adjusted 47pf and 100uf capacitor footprints
Parts:
- C5: footprint Capacitor_THT:C_Radial_D6.3mm_H11.0mm_P2.50mm -> Capacitor_THT:C_Radial_D5.0mm_H11.0mm_P2.00mm
Changed lines of the file:
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@@
 			)
 		)
-		(property "Footprint" "Capacitor_THT:C_Radial_D6.3mm_H11.0mm_P2.50mm"
+		(property "Footprint" "Capacitor_THT:C_Radial_D5.0mm_H11.0mm_P2.00mm"
 			(at 147.32 86.36 0)
 			(hide yes)
