File: Fury-Taur.kicad_sch (KiCad schematic)
At the start: 26 parts, among them J1 Pickup, J2 Output, J3 Audio Out, Q1 J201, Q2 J201, SW1 Push Pull, SW2 SW_SPDT

Commit message: Made single library entry for Push Pull Switch. Updated schematic and PCB with the entry
Parts:
- removed RV1: Volume, symbol Device:R_Potentiometer_US
- removed SW1: Push Pull, symbol Switch:SW_Slide_DPDT
- added RV1: (no value), Custom:PushPull_Pot_DPDT, symbol CustomSymbols:PushPull_Pot_DPDT
Connections:
- net GND: now also RV1.10 (Case), RV1.3 (CW)
- net at J1.5 (Pin_5): now also RV1.1 (CCW)
- net at J2.1 (Pin_1), J3.T: now also RV1.8 (B-Com)
- net at C1.2: now also RV1.4 (A1)
- net at R5.2: now also RV1.7 (B1)
- new net: RV1.2 (Wiper), RV1.5 (A-Com)
- new net: RV1.6 (A2), RV1.9 (B2)
Other:
- company: (none) -> Disco3
- title: (none) -> Fury-Taur
Changed lines of the file:
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@@
 	(generator_version "10.0")
 	(paper "A4")
+	(title_block
+		(title "Fury-Taur")
+		(company "Disco3")
+	)
 	(junction
 		(at 195.58 146.05)
@@
 	(junction
 		(at 142.24 146.05)
+		(diameter 0)
+		(color 0 0 0 0)
+	)
+	(junction
+		(at 88.9 91.44)
 		(diameter 0)
 		(color 0 0 0 0)
@@
 	(wire
 		(pts
+			(xy 88.9 91.44) (xy 88.9 85.09)
+		)
+		(stroke
+			(width 0)
+			(type default)
+		)
+	)
+	(wire
+		(pts
 			(xy 160.02 92.71) (xy 165.1 92.71)
 		)
@@
 	(wire
 		(pts
+			(xy 88.9 91.44) (xy 97.79 91.44)
+		)
+		(stroke
+			(width 0)
+			(type default)
+		)
+	)
+	(wire
+		(pts
 			(xy 165.1 92.71) (xy 172.72 92.71)
 		)
@@
 	(wire
 		(pts
-			(xy 88.9 146.05) (xy 88.9 85.09)
+			(xy 88.9 146.05) (xy 88.9 91.44)
 		)
 		(stroke
@@
 	)
 	(symbol
-		(lib_id "Device:R_Potentiometer_US")
-		(at 101.6 85.09 270)
-		(unit 1)
-		(body_style 1)
-		(exclude_from_sim no)
-		(in_bom yes)
-		(on_board yes)
-		(in_pos_files yes)
-		(dnp no)
-		(fields_autoplaced yes)
-		(property "Reference" "RV1"
-			(at 101.6 78.74 90)
-			(show_name no)
-			(do_not_autoplace no)
-			(effects
-				(font
-					(size 1.27 1.27)
-				)
-			)
-		)
-		(property "Value" "Volume"
-			(at 101.6 81.28 90)
-			(show_name no)
-			(do_not_autoplace no)
-			(effects
-				(font
-					(size 1.27 1.27)
-				)
-			)
-		)
-		(property "Footprint" ""
-			(at 101.6 85.09 0)
-			(hide yes)
-			(show_name no)
-			(do_not_autoplace no)
-			(effects
-				(font
-					(size 1.27 1.27)
-				)
-			)
-		)
-		(property "Datasheet" ""
-			(at 101.6 85.09 0)
-			(hide yes)
-			(show_name no)
-			(do_not_autoplace no)
-			(effects
-				(font
-					(size 1.27 1.27)
-				)
-			)
-		)
-		(property "Description" "Potentiometer, US symbol"
-			(at 101.6 85.09 0)
-			(hide yes)
-			(show_name no)
-			(do_not_autoplace no)
-			(effects
-				(font
-					(size 1.27 1.27)
-				)
-			)
-		)
-		(property "Sim.Device" "R"
-			(at 101.6 85.09 0)
-			(hide yes)
-			(show_name no)
-			(do_not_autoplace no)
-			(effects
-				(font
-					(size 1.27 1.27)
-				)
-			)
-		)
-		(property "Sim.Type" "POT"
-			(at 101.6 85.09 0)
-			(hide yes)
-			(show_name no)
-			(do_not_autoplace no)
-			(effects
-				(font
-					(size 1.27 1.27)
-				)
-			)
-		)
-		(property "Sim.Pins" "1=r0 2=wiper 3=r1"
-			(at 101.6 85.09 0)
-			(hide yes)
-			(show_name no)
-			(do_not_autoplace no)
-			(effects
-				(font
-					(size 1.27 1.27)
-				)
-			)
-		)
-		(pin "3"
-		)
-		(pin "2"
-		)
-		(pin "1"
-		)
-		(instances
-			(project "Mino-Taur"
-				(path "/0fa53c00-8b42-4dbc-a273-f7f4a67fced0"
-					(reference "RV1")
-					(unit 1)
-				)
-			)
-			(project "Fury-Taur"
-				(path "/9aaae789-b710-4a8a-aadd-535a824b9702"
-					(reference "RV1")
-					(unit 1)
-				)
-			)
-		)
-	)
-	(symbol
 		(lib_id "Connector:Screw_Terminal_01x03")
 		(at 215.9 143.51 0)
@@
 				(path "/9aaae789-b710-4a8a-aadd-535a824b9702"
 					(reference "J2")
-					(unit 1)
-				)
-			)
-		)
-	)
-	(symbol
-		(lib_id "Switch:SW_Slide_DPDT")
-		(at 101.6 121.92 0)
-		(unit 1)
-		(body_style 1)
-		(exclude_from_sim no)
-		(in_bom yes)
-		(on_board yes)
-		(in_pos_files yes)
-		(dnp no)
-		(fields_autoplaced yes)
-		(property "Reference" "SW1"
-			(at 101.6 111.76 0)
-			(show_name no)
-			(do_not_autoplace no)
-			(effects
-				(font
-					(size 1.27 1.27)
-				)
-			)
-		)
-		(property "Value" "Push Pull"
-			(at 101.6 114.3 0)
-			(show_name no)
-			(do_not_autoplace no)
-			(effects
-				(font
-					(size 1.27 1.27)
-				)
-			)
-		)
-		(property "Footprint" ""
-			(at 115.57 116.84 0)
-			(hide yes)
-			(show_name no)
-			(do_not_autoplace no)
-			(effects
-				(font
-					(size 1.27 1.27)
-				)
-			)
-		)
-		(property "Datasheet" ""
-			(at 101.6 121.92 0)
-			(hide yes)
-			(show_name no)
-			(do_not_autoplace no)
-			(effects
-				(font
-					(size 1.27 1.27)
-				)
-			)
-		)
-		(property "Description" "Slide Switch, dual pole double throw"
-			(at 101.6 121.92 0)
-			(hide yes)
-			(show_name no)
-			(do_not_autoplace no)
-			(effects
-				(font
-					(size 1.27 1.27)
-				)
-			)
-		)
-		(pin "5"
-		)
-		(pin "6"
-		)
-		(pin "4"
-		)
-		(pin "3"
-		)
-		(pin "2"
-		)
-		(pin "1"
-		)
-		(instances
-			(project "Mino-Taur"
-				(path "/0fa53c00-8b42-4dbc-a273-f7f4a67fced0"
-					(reference "SW1")
-					(unit 1)
-				)
-			)
-			(project "Fury-Taur"
-				(path "/9aaae789-b710-4a8a-aadd-535a824b9702"
-					(reference "SW1")
 					(unit 1)
 				)
@@
 	)
 	(symbol
+		(lib_id "CustomSymbols:PushPull_Pot_DPDT")
+		(at 101.6 119.38 0)
+		(unit 2)
+		(body_style 1)
+		(exclude_from_sim no)
+		(in_bom yes)
+		(on_board yes)
+		(in_pos_files yes)
+		(dnp no)
+		(fields_autoplaced yes)
+		(property "Reference" "RV1"
+			(at 101.6 131.318 0)
+			(show_name no)
+			(do_not_autoplace no)
+			(effects
+				(font
+					(size 1.27 1.27)
+				)
+			)
+		)
+		(property "Value" ""
+			(at 101.6 119.38 0)
+			(hide yes)
+			(show_name no)
+			(do_not_autoplace no)
+			(effects
+				(font
+					(size 1.27 1.27)
+				)
+			)
+		)
+		(property "Footprint" "Custom:PushPull_Pot_DPDT"
+			(at 101.6 113.538 0)
+			(hide yes)
+			(show_name no)
+			(do_not_autoplace no)
+			(effects
+				(font
+					(size 1.27 1.27)
+				)
+			)
+		)
+		(property "Datasheet" ""
+			(at 101.6 119.38 0)
+			(hide yes)
+			(show_name no)
+			(do_not_autoplace no)
+			(effects
+				(font
+					(size 1.27 1.27)
+				)
+			)
+		)
+		(property "Description" ""
+			(at 101.6 119.38 0)
+			(hide yes)
+			(show_name no)
+			(do_not_autoplace no)
+			(effects
+				(font
+					(size 1.27 1.27)
+				)
+			)
+		)
+		(pin "2"
+		)
+		(pin "1"
+		)
+		(pin "6"
+		)
+		(pin "8"
+		)
+		(pin "7"
+		)
+		(pin "9"
+		)
+		(pin "3"
+		)
+		(pin "5"
+		)
+		(pin "10"
+		)
+		(pin "4"
+		)
+		(instances
+			(project "Fury-Taur"
+				(path "/9aaae789-b710-4a8a-aadd-535a824b9702"
+					(reference "RV1")
+					(unit 2)
+				)
+			)
+		)
+	)
+	(symbol
 		(lib_id "Device:D")
 		(at 172.72 129.54 90)
@@
 					(unit 1)
 				)
+			)
+		)
+	)
+	(symbol
+		(lib_id "CustomSymbols:PushPull_Pot_DPDT")
+		(at 101.6 85.09 0)
+		(unit 1)
+		(body_style 1)
+		(exclude_from_sim no)
+		(in_bom yes)
+		(on_board yes)
+		(in_pos_files yes)
+		(dnp no)
+		(fields_autoplaced yes)
+		(property "Reference" "RV1"
+			(at 101.6 97.028 0)
+			(show_name no)
+			(do_not_autoplace no)
+			(effects
+				(font
+					(size 1.27 1.27)
+				)
+			)
+		)
+		(property "Value" ""
+			(at 101.6 85.09 0)
+			(hide yes)
+			(show_name no)
+			(do_not_autoplace no)
+			(effects
+				(font
+					(size 1.27 1.27)
+				)
+			)
+		)
+		(property "Footprint" "Custom:PushPull_Pot_DPDT"
+			(at 101.6 79.248 0)
+			(hide yes)
+			(show_name no)
+			(do_not_autoplace no)
+			(effects
+				(font
+					(size 1.27 1.27)
+				)
+			)
+		)
+		(property "Datasheet" ""
+			(at 101.6 85.09 0)
+			(hide yes)
+			(show_name no)
+			(do_not_autoplace no)
+			(effects
+				(font
+					(size 1.27 1.27)
+				)
+			)
+		)
+		(property "Description" ""
+			(at 101.6 85.09 0)
+			(hide yes)
+			(show_name no)
+			(do_not_autoplace no)
+			(effects
+				(font
+					(size 1.27 1.27)
+				)
+			)
+		)
+		(pin "2"
+		)
+		(pin "1"
+		)
+		(pin "6"
+		)
+		(pin "8"
+		)
+		(pin "7"
+		)
+		(pin "9"
+		)
+		(pin "3"
+		)
+		(pin "5"
+		)
+		(pin "10"
+		)
+		(pin "4"
+		)
+		(instances
+			(project "Fury-Taur"
+				(path "/9aaae789-b710-4a8a-aadd-535a824b9702"
+					(reference "RV1")
+					(unit 1)
+				)

Commit message: Updated various behind the scenes things, such as C5 polarazed symbol, J201 datasheet, add #PWR_FLAG to power
Parts:
- C2, C7: footprint Capacitor_THT:C_Disc_D5.1mm_W3.2mm_P5.00mm -> Capacitor_THT:C_Disc_D4.7mm_W2.5mm_P5.00mm
- C5: symbol Device:C_US -> Device:C_Polarized_US
- D1: footprint Diode_THT:D_DO-35_SOD27_P10.16mm_Horizontal -> Diode_THT:D_DO-41_SOD81_P10.16mm_Horizontal
- J1: footprint TerminalBlock_4Ucon:TerminalBlock_4Ucon_1x05_P3.50mm_Horizontal -> TerminalBlock_Phoenix:TerminalBlock_Phoenix_PT-1,5-5-3.5-H_1x05_P3.50mm_Horizontal
- J2: footprint TerminalBlock_4Ucon:TerminalBlock_4Ucon_1x03_P3.50mm_Horizontal -> TerminalBlock_Phoenix:TerminalBlock_Phoenix_PT-1,5-3-3.5-H_1x03_P3.50mm_Horizontal
Connections:
- net at C2.1, C5.1, C7.1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: now also RV2.1, RV3.1; no longer RV2.3, RV3.3
- net at C6.2, C7.2, Q2.1 (D): now also RV3.3; no longer RV3.1
- net at C2.2, C3.2, Q1.1 (D): now also RV2.3; no longer RV2.1
Changed lines of the file:
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@@
 	)
 	(junction
+		(at 138.43 76.2)
+		(diameter 0)
+		(color 0 0 0 0)
+	)
+	(junction
 		(at 173.99 146.05)
 		(diameter 0)
@@
 	)
 	(junction
+		(at 199.39 143.51)
+		(diameter 0)
+		(color 0 0 0 0)
+	)
+	(junction
 		(at 130.81 105.41)
 		(diameter 0)
@@
 	(wire
 		(pts
+			(xy 138.43 76.2) (xy 135.89 76.2)
+		)
+		(stroke
+			(width 0)
+			(type default)
+		)
+	)
+	(wire
+		(pts
 			(xy 88.9 85.09) (xy 97.79 85.09)
 		)
@@
 	(wire
 		(pts
-			(xy 139.7 76.2) (xy 135.89 76.2)
+			(xy 139.7 76.2) (xy 138.43 76.2)
 		)
 		(stroke
@@
 	)
 	(symbol
+		(lib_id "power:PWR_FLAG")
+		(at 199.39 143.51 0)
+		(unit 1)
+		(body_style 1)
+		(exclude_from_sim no)
+		(in_bom yes)
+		(on_board yes)
+		(in_pos_files yes)
+		(dnp no)
+		(fields_autoplaced yes)
+		(property "Reference" "#FLG02"
+			(at 199.39 141.605 0)
+			(hide yes)
+			(show_name no)
+			(do_not_autoplace no)
+			(effects
+				(font
+					(size 1.27 1.27)
+				)
+			)
+		)
+		(property "Value" "PWR_FLAG"
+			(at 199.39 138.43 0)
+			(show_name no)
+			(do_not_autoplace no)
+			(effects
+				(font
+					(size 1.27 1.27)
+				)
+			)
+		)
+		(property "Footprint" ""
+			(at 199.39 143.51 0)
+			(hide yes)
+			(show_name no)
+			(do_not_autoplace no)
+			(effects
+				(font
+					(size 1.27 1.27)
+				)
+			)
+		)
+		(property "Datasheet" ""
+			(at 199.39 143.51 0)
+			(hide yes)
+			(show_name no)
+			(do_not_autoplace no)
+			(effects
+				(font
+					(size 1.27 1.27)
+				)
+			)
+		)
+		(property "Description" "Special symbol for telling ERC where power comes from"
+			(at 199.39 143.51 0)
+			(hide yes)
+			(show_name no)
+			(do_not_autoplace no)
+			(effects
+				(font
+					(size 1.27 1.27)
+				)
+			)
+		)
+		(pin "1"
+		)
+		(instances
+			(project "Fury-Taur"
+				(path "/9aaae789-b710-4a8a-aadd-535a824b9702"
+					(reference "#FLG02")
+					(unit 1)
+				)
+			)
+		)
+	)
+	(symbol
+		(lib_id "power:PWR_FLAG")
+		(at 138.43 76.2 0)
+		(unit 1)
+		(body_style 1)
+		(exclude_from_sim no)
+		(in_bom yes)
+		(on_board yes)
+		(in_pos_files yes)
+		(dnp no)
+		(fields_autoplaced yes)
+		(property "Reference" "#FLG01"
+			(at 138.43 74.295 0)
+			(hide yes)
+			(show_name no)
+			(do_not_autoplace no)
+			(effects
+				(font
+					(size 1.27 1.27)
+				)
+			)
+		)
+		(property "Value" "PWR_FLAG"
+			(at 138.43 71.12 0)
+			(show_name no)
+			(do_not_autoplace no)
+			(effects
+				(font
+					(size 1.27 1.27)
+				)
+			)
+		)
+		(property "Footprint" ""
+			(at 138.43 76.2 0)
+			(hide yes)
+			(show_name no)
+			(do_not_autoplace no)
+			(effects
+				(font
+					(size 1.27 1.27)
+				)
+			)
+		)
+		(property "Datasheet" ""
+			(at 138.43 76.2 0)
+			(hide yes)
+			(show_name no)
+			(do_not_autoplace no)
+			(effects
+				(font
+					(size 1.27 1.27)
+				)
+			)
+		)
+		(property "Description" "Special symbol for telling ERC where power comes from"
+			(at 138.43 76.2 0)
+			(hide yes)
+			(show_name no)
+			(do_not_autoplace no)
+			(effects
+				(font
+					(size 1.27 1.27)
+				)
+			)
+		)
+		(pin "1"
+		)
+		(instances
+			(project "Fury-Taur"
+				(path "/9aaae789-b710-4a8a-aadd-535a824b9702"
+					(reference "#FLG01")
+					(unit 1)
+				)
+			)
+		)
+	)
+	(symbol
 		(lib_id "power:GND")
 		(at 199.39 152.4 0)
@@
 			)
 		)
-		(property "Footprint" "Diode_THT:D_DO-35_SOD27_P10.16mm_Horizontal"
+		(property "Footprint" "Diode_THT:D_DO-41_SOD81_P10.16mm_Horizontal"
 			(at 143.51 76.2 0)
 			(hide yes)
@@
 			)
 		)
-		(property "Footprint" "TerminalBlock_4Ucon:TerminalBlock_4Ucon_1x03_P3.50mm_Horizontal"
+		(property "Footprint" "TerminalBlock_Phoenix:TerminalBlock_Phoenix_PT-1,5-3-3.5-H_1x03_P3.50mm_Horizontal"
 			(at 215.9 143.51 0)
 			(hide yes)
@@
 			)
 		)
-		(property "Datasheet" "https://www.onsemi.com/pub/Collateral/MMBFJ113-D.PDF"
+		(property "Datasheet" "https://www.interfet.com/jfet-datasheets/jfet-j201-j202-interfet.pdf"
 			(at 162.56 114.3 0)
 			(hide yes)
@@
 	)
 	(symbol
-		(lib_name "R_Potentiometer_Trim_US_1")
 		(lib_id "Device:R_Potentiometer_Trim_US")
 		(at 115.57 86.36 0)
@@
 	)
 	(symbol
-		(lib_id "Device:C_US")
+		(lib_id "Device:C_Polarized_US")
 		(at 147.32 86.36 0)
 		(unit 1)
@@
 		(fields_autoplaced yes)
 		(property "Reference" "C5"
-			(at 151.13 85.3439 0)
+			(at 151.13 84.4549 0)
 			(show_name no)
 			(do_not_autoplace no)
@@
 		)
 		(property "Value" "100uf"
-			(at 151.13 87.8839 0)
+			(at 151.13 86.9949 0)
 			(show_name no)
 			(do_not_autoplace no)
@@
 			)
 		)
-		(property "Description" "capacitor, US symbol"
+		(property "Description" "Polarized capacitor, US symbol"
 			(at 147.32 86.36 0)
 			(hide yes)
@@
 			)
 		)
-		(property "Footprint" "Capacitor_THT:C_Disc_D5.1mm_W3.2mm_P5.00mm"
+		(property "Footprint" "Capacitor_THT:C_Disc_D4.7mm_W2.5mm_P5.00mm"
 			(at 124.1552 90.17 0)
 			(hide yes)
@@
 			)
 		)
-		(property "Footprint" "Capacitor_THT:C_Disc_D5.1mm_W3.2mm_P5.00mm"
+		(property "Footprint" "Capacitor_THT:C_Disc_D4.7mm_W2.5mm_P5.00mm"
 			(at 173.6852 90.17 0)
 			(hide yes)
@@
 	)
 	(symbol
-		(lib_name "R_Potentiometer_Trim_US_2")
 		(lib_id "Device:R_Potentiometer_Trim_US")
 		(at 165.1 86.36 0)
@@
 			)
 		)
-		(property "Datasheet" "https://www.onsemi.com/pub/Collateral/MMBFJ113-D.PDF"
+		(property "Datasheet" "https://www.interfet.com/jfet-datasheets/jfet-j201-j202-interfet.pdf"
 			(at 133.35 120.65 0)
 			(hide yes)
@@
 			)
 		)
-		(property "Footprint" "TerminalBlock_4Ucon:TerminalBlock_4Ucon_1x05_P3.50mm_Horizontal"
+		(property "Footprint" "TerminalBlock_Phoenix:TerminalBlock_Phoenix_PT-1,5-5-3.5-H_1x05_P3.50mm_Horizontal"
 			(at 74.93 97.79 0)
 			(hide yes)

Commit message: Updated various behind the scenes things, such as C5 polarazed symbol, J201 datasheet, add #PWR_FLAG to power
Parts:
- C5: footprint Capacitor_THT:C_Radial_D5.0mm_H11.0mm_P2.00mm -> Capacitor_THT:CP_Radial_D5.0mm_P2.00mm
Changed lines of the file:
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@@
 			)
 		)
-		(property "Description" "2mA min, 35V, 100mOhm max, 0.5-3V Vgs(off), N-Channel JFET, SOT-23"
+		(property "Description" "J201 N-channel JFET, TO-92"
 			(at 157.48 110.49 0)
 			(hide yes)
@@
 			)
 		)
-		(property "Footprint" "Capacitor_THT:C_Radial_D5.0mm_H11.0mm_P2.00mm"
+		(property "Footprint" "Capacitor_THT:CP_Radial_D5.0mm_P2.00mm"
 			(at 147.32 86.36 0)
 			(hide yes)
@@
 			)
 		)
-		(property "Description" "2mA min, 35V, 100mOhm max, 0.5-3V Vgs(off), N-Channel JFET, SOT-23"
+		(property "Description" "J201 N-channel JFET, TO-92"
 			(at 128.27 116.84 0)
 			(hide yes)

Commit message: Re-Annotated components
Parts:
- J3, L1, L2: now left out of the parts list
- renumbered C5 to C4, C6 to C5, C7 to C6, R4 to R3, R3 to RV4, R5 to RV5, SW2 to SW1
Changed lines of the file:
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@@
 		(property "Value" "PWR_FLAG"
 			(at 199.39 138.43 0)
+			(hide yes)
 			(show_name no)
 			(do_not_autoplace no)
@@
 		(property "Value" "PWR_FLAG"
 			(at 138.43 71.12 0)
+			(hide yes)
 			(show_name no)
 			(do_not_autoplace no)
@@
 		(dnp no)
 		(fields_autoplaced yes)
-		(property "Reference" "#PWR05"
+		(property "Reference" "#PWR06"
 			(at 199.39 158.75 0)
 			(hide yes)
@@
 			(project "Fury-Taur"
 				(path "/9aaae789-b710-4a8a-aadd-535a824b9702"
-					(reference "#PWR05")
+					(reference "#PWR06")
 					(unit 1)
 				)
@@
 		(body_style 1)
 		(exclude_from_sim no)
-		(in_bom yes)
+		(in_bom no)
 		(on_board no)
 		(in_pos_files yes)
@@
 		(dnp no)
 		(fields_autoplaced yes)
-		(property "Reference" "R4"
+		(property "Reference" "R3"
 			(at 172.72 96.52 90)
 			(show_name no)
@@
 			)
 		)
-		(property "Datasheet" "14"
+		(property "Datasheet" ""
 			(at 172.72 102.87 0)
 			(hide yes)
@@
 			(project "Fury-Taur"
 				(path "/9aaae789-b710-4a8a-aadd-535a824b9702"
-					(reference "R4")
+					(reference "R3")
 					(unit 1)
 				)
@@
 		(body_style 1)
 		(exclude_from_sim no)
-		(in_bom yes)
+		(in_bom no)
 		(on_board no)
 		(in_pos_files yes)
@@
 		(dnp no)
 		(fields_autoplaced yes)
-		(property "Reference" "R3"
+		(property "Reference" "RV4"
 			(at 143.51 109.2199 0)
 			(show_name no)
@@
 			(project "Fury-Taur"
 				(path "/9aaae789-b710-4a8a-aadd-535a824b9702"
-					(reference "R3")
+					(reference "RV4")
 					(unit 1)
 				)
@@
 		(body_style 1)
 		(exclude_from_sim no)
-		(in_bom yes)
+		(in_bom no)
 		(on_board no)
 		(in_pos_files yes)
@@
 		(dnp no)
 		(fields_autoplaced yes)
-		(property "Reference" "#PWR04"
+		(property "Reference" "#PWR05"
 			(at 147.32 96.52 0)
 			(hide yes)
@@
 			(project "Fury-Taur"
 				(path "/9aaae789-b710-4a8a-aadd-535a824b9702"
-					(reference "#PWR04")
+					(reference "#PWR05")
 					(unit 1)
 				)
@@
 		(dnp no)
 		(fields_autoplaced yes)
-		(property "Reference" "C5"
+		(property "Reference" "C4"
 			(at 151.13 84.4549 0)
 			(show_name no)
@@
 			(project "Fury-Taur"
 				(path "/9aaae789-b710-4a8a-aadd-535a824b9702"
-					(reference "C5")
+					(reference "C4")
 					(unit 1)
 				)
@@
 		(dnp no)
 		(fields_autoplaced yes)
-		(property "Reference" "#PWR06"
+		(property "Reference" "#PWR03"
 			(at 88.9 152.4 0)
 			(hide yes)
@@
 			(project "Fury-Taur"
 				(path "/9aaae789-b710-4a8a-aadd-535a824b9702"
-					(reference "#PWR06")
+					(reference "#PWR03")
 					(unit 1)
 				)
@@
 		(in_pos_files yes)
 		(dnp no)
-		(property "Reference" "SW2"
+		(property "Reference" "SW1"
 			(at 177.8 107.95 0)
 			(show_name no)
@@
 			(project "Fury-Taur"
 				(path "/9aaae789-b710-4a8a-aadd-535a824b9702"
-					(reference "SW2")
+					(reference "SW1")
 					(unit 1)
 				)
@@
 		(dnp no)
 		(fields_autoplaced yes)
-		(property "Reference" "C7"
+		(property "Reference" "C6"
 			(at 176.53 85.0899 0)
 			(show_name no)
@@
 			(project "Fury-Taur"
 				(path "/9aaae789-b710-4a8a-aadd-535a824b9702"
-					(reference "C7")
+					(reference "C6")
 					(unit 1)
 				)
@@
 		(dnp no)
 		(fields_autoplaced yes)
-		(property "Reference" "#PWR03"
+		(property "Reference" "#PWR04"
 			(at 135.89 80.01 0)
 			(hide yes)
@@
 			(project "Fury-Taur"
 				(path "/9aaae789-b710-4a8a-aadd-535a824b9702"
-					(reference "#PWR03")
+					(reference "#PWR04")
 					(unit 1)
 				)
@@
 		(dnp no)
 		(fields_autoplaced yes)
-		(property "Reference" "R5"
+		(property "Reference" "RV5"
 			(at 193.04 105.4099 0)
 			(show_name no)
@@
 			(project "Fury-Taur"
 				(path "/9aaae789-b710-4a8a-aadd-535a824b9702"
-					(reference "R5")
+					(reference "RV5")
 					(unit 1)
 				)
@@
 		(dnp no)
 		(fields_autoplaced yes)
-		(property "Reference" "C6"
+		(property "Reference" "C5"
 			(at 163.83 95.25 90)
 			(show_name no)
@@
 			(project "Fury-Taur"
 				(path "/9aaae789-b710-4a8a-aadd-535a824b9702"
-					(reference "C6")
-					(unit 1)
-				)
+					(reference "C5")
+					(unit 1)
+				)
