File: ~gerberzipper_temp/Fury-Taur.kicad_pcb (KiCad board)
At the start: 2 copper layers, 75.1 x 26.5 mm, 31 parts, among them J1 Pickup, J2 Output, Q1 Bias 20K, Q1 J201, Q1 Test TestPoint_THTPad_1.0x1.0mm_Dr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, Q2 Bias 20K, Q2 J201, Q2 Test TestPoint_THTPad_1.0x1.0mm_Dr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, SW1 ALPHA_PUSH_PULL, SW2 SW_SPDT

Commit message: Labeled test pads, reworked front silkscreen
Other:
- board text removed: "100μF"
- board text removed: "47pf"
- board text removed: "Gain"
- board text removed: "J201"
- board text removed: "Level"
Changed lines of the file:
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@@
-		)
-	)
-	(gr_text "100μF"
-		(at 105.52 80.25 0)
-		(layer "F.SilkS")
-		(effects
-			(font
-				(size 0.72 0.72)
-				(thickness 0.108)
-			)
 		)
 	)
@@
 		)
 	)
-	(gr_text "47pf"
-		(at 118.5 78 0)
-		(layer "F.SilkS")
-		(effects
-			(font
-				(size 0.72 0.72)
-				(thickness 0.108)
-			)
-		)
-	)
 	(gr_text "Q2"
 		(at 123.77 67.5 0)
-		(layer "F.SilkS")
-		(effects
-			(font
-				(size 0.72 0.72)
-				(thickness 0.108)
-			)
-		)
-	)
-	(gr_text "47pf"
-		(at 130 78 0)
 		(layer "F.SilkS")
 		(effects
@@
 		)
 	)
-	(gr_text "J201"
-		(at 116.229 70.29 0)
-		(layer "F.SilkS")
-		(effects
-			(font
-				(size 1 1)
-				(thickness 0.15)
-			)
-		)
-	)
 	(gr_text "C2"
 		(at 118.5 80.5 0)
@@
 	(gr_text "C6"
 		(at 118.7 75 0)
-		(layer "F.SilkS")
-		(effects
-			(font
-				(size 1 1)
-				(thickness 0.15)
-			)
-		)
-	)
-	(gr_text "J201"
-		(at 123.77 70.29 0)
 		(layer "F.SilkS")
 		(effects
@@
 		(layer "F.SilkS")
 		(effects
-			(font
-				(size 1 1)
-				(thickness 0.15)
-			)
-		)
-	)
-	(gr_text "Gain"
-		(at 132.34 69.67 0)
-		(layer "F.SilkS")
-		(effects
-			(font
-				(size 1 1)
-				(thickness 0.15)
-			)
-		)
-	)
-	(gr_text "Level"
-		(at 143.14 69.67 0)
-		(layer "F.SilkS")
-		(effects
